Commit message: Add real-physics Gazebo variant with real object spawning
Extends demo_gazebo.launch.py from a booting-but-blocked sim into a fully
working real-physics run for both variants:

- Root-caused and fixed the MoveIt/Gazebo clock mismatch (moveit2#2940):
  remap the gz_ros2_control plugin's raw joint states to /joint_states_raw
  in the xacro, and have joint_state_restamp.py republish them wall-clock
  stamped on /joint_states, the name everything else already expects.
- Anchored the robot base to the world with a real fixed joint in
  panda_gazebo.urdf.xacro (the upstream URDF only had a MoveIt-only SRDF
  virtual joint, invisible to Gazebo physics - the arm fell over).
- Widened allowed_start_tolerance for real settling lag mock hardware never
  has, and tuned position_proportional_gain in a new
  ros2_controllers_gazebo.yaml for gz_ros_control's position interface.
- Found and fixed three separate startup-race conditions in sequence (fixed
  delay -> action-list poll -> add a /joint_states-flowing check), each a
  distinct DDS discovery-timing gap exposed only once the previous one was
  fixed.
- Added gazebo_scene_adapter.py so every recipe part/obstacle is spawned as
  a real physical Gazebo model (not just MoveIt/RViz planning-scene
  geometry), composed alongside the existing MoveIt scene adapter via
  CompositeSceneAdapter - the MoveIt path is unchanged, this only adds to
  it.

Verified live for both variants: Approach and Pick plan, execute under real
gravity/contact and verify successfully; Retreat correctly hits the same
genuine keepout collision as the mock-hardware run, driving the same
recovery sequence. Full account with live evidence in
docs/moveit2_integration_notes.md.

File: config/panda_gazebo.urdf.xacro (robot description, xacro)
@@ -14,5 +14,20 @@
 -->
 <robot xmlns:xacro="http://www.ros.org/wiki/xacro" name="panda">
+  <xacro:arg name="controllers_config_path"
+             default="$(find moveit_resources_panda_moveit_config)/config/ros2_controllers.yaml" />
   <xacro:include filename="$(find moveit_resources_panda_description)/urdf/panda.urdf.xacro" />
+  <!-- moveit_resources_panda_description's URDF has no joint at all
+       anchoring panda_link0 to anything - the SRDF's virtual_joint (world ->
+       panda_link0, type "floating") is a MoveIt-only planning construct with
+       no effect on Gazebo physics. Under mock_components (no physics) this
+       is invisible; under real gravity the whole robot is an unanchored free
+       body and topples over (confirmed live). Fix: a real fixed joint,
+       matching astra_ros.tf_adapter's WORLD_TO_BASE identity assumption. -->
+  <link name="world"/>
+  <joint name="world_to_panda_link0" type="fixed">
+    <parent link="world"/>
+    <child link="panda_link0"/>
+    <origin xyz="0 0 0" rpy="0 0 0"/>
+  </joint>
   <ros2_control name="PandaGazeboSystem" type="system">
     <hardware>
@@ -66,5 +81,14 @@
   <gazebo>
     <plugin filename="gz_ros2_control-system" name="gz_ros2_control::GazeboSimROS2ControlPlugin">
-      <parameters>$(find moveit_resources_panda_moveit_config)/config/ros2_controllers.yaml</parameters>
+      <parameters>$(arg controllers_config_path)</parameters>
+      <!-- Remap the raw (simulated-time-stamped) joint_states off its default
+           name so astra_ros.nodes.joint_state_restamp can own the name
+           "/joint_states" instead - see docs/moveit2_integration_notes.md
+           ("Gazebo (gz_sim) physics simulation") for why MoveItPy's
+           CurrentStateMonitor cannot itself be redirected to a renamed
+           topic. -->
+      <ros>
+        <remapping>/joint_states:=/joint_states_raw</remapping>
+      </ros>
     </plugin>
   </gazebo>
